Commit message: darwin updates

File: catkin_ws/src/hardware/darwin/darwin_description/urdf/darwin_lab.urdf (robot description, URDF)
Before this commit: robot darwin_lab, 31 links, 30 joints
Links:
- added link imu_link
Joints:
- added joint imu: type fixed, parent base_link, child imu_link, origin xyz=0 0 0 rpy=0 0 0

Commit message: fixed luckfox camera, close #23

File: catkin_ws/src/hardware/darwin/darwin_description/urdf/darwin_lab.urdf (robot description, URDF)
Before this commit: robot darwin_lab, 32 links, 31 joints
Links:
- link camera_optical: geometry visual box size=0.032 0.005 0.032

Commit message: finally darwin has right frames on both feet

File: catkin_ws/src/hardware/darwin/darwin_description/urdf/darwin_lab.urdf (robot description, URDF)
Before this commit: robot darwin_lab, 32 links, 31 joints
Joints:
- joint imu: parent base_link -> trunk_link
- joint left_ankle_roll: axis 0 0 1 -> 1 0 0; origin xyz=0 0 0 rpy=-1.5707963 0 0 -> xyz=0 0 0 rpy=1.5707 0 1.5707
- joint right_ankle_roll: axis 0 0 1 -> 1 0 0; origin xyz=0 0 0 rpy=-1.5707963 0 0 -> xyz=0 0 0 rpy=-1.5707 0 1.5707

Commit message: URDF DARWIN CORRECT JOINT FRAMES

File: catkin_ws/src/hardware/darwin/darwin_description/urdf/darwin_lab.urdf (robot description, URDF)
Before this commit: robot darwin_lab, 32 links, 31 joints
Links:
- link MP_ARM_GRIPPER_MOV_R: geometry collision box size=0.032 0.005 0.032; visual box size=0.032 0.005 0.032
Joints:
- joint camera_joint: axis 0 0 1 -> (none); limit lower=-2.6179939 upper=2.6179939 effort=2.8 velocity=5.6548668 -> (none); origin xyz=0 0 0.0235 rpy=3.14159 1.5707963 0 -> xyz=0 0 0.0235 rpy=0 0 0
- joint head_pitch: axis 0 0 1 -> 0 1 0; origin xyz=0 0 0.02715 rpy=-1.5707963 0 1.5707963 -> xyz=0 0 0.02715 rpy=0 0 0
- joint j_back_l: origin xyz=0 0.06035 0 rpy=-1.5707963 0 0 -> xyz=0 0.06035 0 rpy=0 0 0
- joint j_back_r: limit lower=-2.6179939 upper=2.6179939 effort=2.8 velocity=5.6548668 -> (none); origin xyz=0 -0.06035 0 rpy=1.5707963 0 0 -> xyz=0 -0.06035 0 rpy=0 0 0
- joint j_gripper_l: axis 0 0 1 -> (none); limit lower=-2.6179939 upper=2.6179939 effort=2.8 velocity=5.6548668 -> (none); origin xyz=0.048 0.01 0 rpy=0 0 1.0 -> xyz=0 0.01 -0.01 rpy=0 1.5707963 0
- joint j_gripper_r: axis 0 0 1 -> (none); limit lower=-2.6179939 upper=2.6179939 effort=2.8 velocity=5.6548668 -> (none); origin xyz=0.048 0.01 0 rpy=0 0 1.0 -> xyz=0 -0.006 -0.04 rpy=0 0 0
- joint j_wrist_dummy_l: origin xyz=0.064 -0.01 0 rpy=0 0 0 -> xyz=0 -0.01 -0.03 rpy=0 0 0
- joint j_wrist_dummy_r: origin xyz=0.064 -0.01 0 rpy=0 0 0 -> xyz=0 -0.026 -0.04 rpy=0 0 0
- joint j_wrist_l: axis 0 0 1 -> (none); limit lower=-2.6179939 upper=2.6179939 effort=2.8 velocity=5.6548668 -> (none); origin xyz=0.048 0.016 0 rpy=1.5707963 0 0 -> xyz=0 0.016 -0.048 rpy=0 0 0
- joint j_wrist_r: axis 0 0 1 -> (none); limit lower=-2.6179939 upper=2.6179939 effort=2.8 velocity=5.6548668 -> (none); origin xyz=0.048 -0.016 0 rpy=1.5707963 0 0 -> xyz=0 0.016 -0.048 rpy=0 0 0
- joint left_ankle_pitch: axis 0 0 1 -> 0 1 0; origin xyz=-0.093 0 0 rpy=3.14159 0 0 -> xyz=0 0 -0.093 rpy=0 0 0
- joint left_ankle_roll: origin xyz=0 0 0 rpy=1.5707 0 1.5707 -> xyz=0 0 0 rpy=0 0 0
- joint left_elbow_pitch: axis 0 0 1 -> 0 1 0; origin xyz=-0.06 0 -0.016 rpy=-1.5707963 3.14159 0 -> xyz=0 -0.016 -0.06 rpy=0 0 0
- joint left_hip_pitch: axis 0 0 1 -> 0 1 0; origin xyz=0 0 0 rpy=1.5707963 0 -1.5707963 -> xyz=0 0 0 rpy=0 0 0
- joint left_hip_roll: axis 0 0 1 -> 1 0 0; origin xyz=0 0 0.028652 rpy=1.5707963 0 0 -> xyz=0 0 -0.028652 rpy=0 0 0
- joint left_hip_yaw: origin xyz=-0.005 0.037 -0.09355 rpy=0 3.14159 -1.5707963 -> xyz=-0.005 0.037 -0.09355 rpy=0 0 0
- joint left_knee_pitch: axis 0 0 1 -> 0 1 0; origin xyz=-0.093 0 0 rpy=0 0 0 -> xyz=0 0 -0.093 rpy=0 0 0
- joint left_shoulder_pitch: axis 0 0 1 -> 0 1 0; origin xyz=0 0 0 rpy=0 0 -1.5707963 -> xyz=0 0 0 rpy=0 0 0
- joint left_shoulder_roll: axis 0 0 1 -> 1 0 0; origin xyz=-0.016 0 0.02165 rpy=1.5707963 1.5707963 0 -> xyz=0 0.02165 -0.016 rpy=0 0 0
- joint neck_yaw: origin xyz=0 0 0.0235 rpy=0 0 1.5707963 -> xyz=0 0 0.0235 rpy=0 0 0
- joint right_ankle_pitch: axis 0 0 1 -> 0 1 0; origin xyz=0.093 0 0 rpy=3.14159 0 0 -> xyz=0 0 -0.093 rpy=0 0 0
- joint right_ankle_roll: origin xyz=0 0 0 rpy=-1.5707 0 1.5707 -> xyz=0 0 0 rpy=0 0 0
- joint right_elbow_pitch: axis 0 0 1 -> 0 1 0 ; origin xyz=-0.06 0 0.016 rpy=-1.5707963 3.14159 0 -> xyz=-0.016 0 -0.06  rpy=0 0 0
- joint right_hip_pitch: axis 0 0 1 -> 0 1 0; origin xyz=0 0 0 rpy=1.5707963 0 -1.5707963 -> xyz=0 0 0 rpy=0 0 0
- joint right_hip_roll: axis 0 0 1 -> 1 0 0; origin xyz=0 0 0.028652 rpy=-1.5707963 0 0 -> xyz=0 0 -0.028652 rpy=0 0 0
- joint right_hip_yaw: origin xyz=-0.005 -0.037 -0.09355 rpy=0 3.14159 1.5707963 -> xyz=-0.005 -0.037 -0.09355 rpy=0 0 0
- joint right_knee_pitch: axis 0 0 1 -> 0 1 0; origin xyz=0.093 0 0 rpy=0 0 0 -> xyz=0 0 -0.093 rpy=0 0 0
- joint right_shoulder_pitch: axis 0 0 1 -> 0 1 0; origin xyz=0 0 0 rpy=0 0 -1.5707963 -> xyz=0 0 0 rpy=0 0 0
- joint right_shoulder_roll: axis 0 0 1 -> 1 0 0; origin xyz=0.016 0 0.02165 rpy=-1.5707963 1.5707963 0 -> xyz=0 -0.02165 -0.016 rpy=0 0 0

File: catkin_ws/src/hardware/darwin/darwin_description/urdf/darwin_lab_fixed.urdf (robot description, URDF)
Before this commit: robot darwin_lab, 33 links, 32 joints
Links:
- link MP_ARM_GRIPPER_MOV_R: geometry collision box size=0.032 0.005 0.032; visual box size=0.032 0.005 0.032
- link camera_optical: geometry visual box size=0.032 0.005 0.032
Joints:
- joint camera_joint: axis 0 0 1 -> (none); limit lower=-2.6179939 upper=2.6179939 effort=2.8 velocity=5.6548668 -> (none); origin xyz=0 0 0.0235 rpy=3.14159 1.5707963 0 -> xyz=0 0 0.0235 rpy=0 0 0
- joint head_pitch: axis 0 0 1 -> 0 1 0; origin xyz=0 0 0.02715 rpy=-1.5707963 0 1.5707963 -> xyz=0 0 0.02715 rpy=0 0 0
- joint imu: parent base_link -> trunk_link
- joint j_back_l: origin xyz=0 0.06035 0 rpy=-1.5707963 0 0 -> xyz=0 0.06035 0 rpy=0 0 0
- joint j_back_r: limit lower=-2.6179939 upper=2.6179939 effort=2.8 velocity=5.6548668 -> (none); origin xyz=0 -0.06035 0 rpy=1.5707963 0 0 -> xyz=0 -0.06035 0 rpy=0 0 0
- joint j_gripper_l: axis 0 0 1 -> (none); limit lower=-2.6179939 upper=2.6179939 effort=2.8 velocity=5.6548668 -> (none); origin xyz=0.048 0.01 0 rpy=0 0 1.0 -> xyz=0 0.01 -0.01 rpy=0 1.5707963 0
- joint j_gripper_r: axis 0 0 1 -> (none); limit lower=-2.6179939 upper=2.6179939 effort=2.8 velocity=5.6548668 -> (none); origin xyz=0.048 0.01 0 rpy=0 0 1.0 -> xyz=0 -0.006 -0.04 rpy=0 0 0
- joint j_wrist_dummy_l: origin xyz=0.064 -0.01 0 rpy=0 0 0 -> xyz=0 -0.01 -0.03 rpy=0 0 0
- joint j_wrist_dummy_r: origin xyz=0.064 -0.01 0 rpy=0 0 0 -> xyz=0 -0.026 -0.04 rpy=0 0 0
- joint j_wrist_l: axis 0 0 1 -> (none); limit lower=-2.6179939 upper=2.6179939 effort=2.8 velocity=5.6548668 -> (none); origin xyz=0.048 0.016 0 rpy=1.5707963 0 0 -> xyz=0 0.016 -0.048 rpy=0 0 0
- joint j_wrist_r: axis 0 0 1 -> (none); limit lower=-2.6179939 upper=2.6179939 effort=2.8 velocity=5.6548668 -> (none); origin xyz=0.048 -0.016 0 rpy=1.5707963 0 0 -> xyz=0 0.016 -0.048 rpy=0 0 0
- joint left_ankle_pitch: axis 0 0 1 -> 0 1 0; origin xyz=-0.093 0 0 rpy=3.14159 0 0 -> xyz=0 0 -0.093 rpy=0 0 0
- joint left_ankle_roll: axis 0 0 1 -> 1 0 0; origin xyz=0 0 0 rpy=-1.5707963 0 0 -> xyz=0 0 0 rpy=0 0 0
- joint left_elbow_pitch: axis 0 0 1 -> 0 1 0; origin xyz=-0.06 0 -0.016 rpy=-1.5707963 3.14159 0 -> xyz=0 -0.016 -0.06 rpy=0 0 0
- joint left_hip_pitch: axis 0 0 1 -> 0 1 0; origin xyz=0 0 0 rpy=1.5707963 0 -1.5707963 -> xyz=0 0 0 rpy=0 0 0
- joint left_hip_roll: axis 0 0 1 -> 1 0 0; origin xyz=0 0 0.028652 rpy=1.5707963 0 0 -> xyz=0 0 -0.028652 rpy=0 0 0
- joint left_hip_yaw: origin xyz=-0.005 0.037 -0.09355 rpy=0 3.14159 -1.5707963 -> xyz=-0.005 0.037 -0.09355 rpy=0 0 0
- joint left_knee_pitch: axis 0 0 1 -> 0 1 0; origin xyz=-0.093 0 0 rpy=0 0 0 -> xyz=0 0 -0.093 rpy=0 0 0
- joint left_shoulder_pitch: axis 0 0 1 -> 0 1 0; origin xyz=0 0 0 rpy=0 0 -1.5707963 -> xyz=0 0 0 rpy=0 0 0
- joint left_shoulder_roll: axis 0 0 1 -> 1 0 0; origin xyz=-0.016 0 0.02165 rpy=1.5707963 1.5707963 0 -> xyz=0 0.02165 -0.016 rpy=0 0 0
- joint neck_yaw: origin xyz=0 0 0.0235 rpy=0 0 1.5707963 -> xyz=0 0 0.0235 rpy=0 0 0
- joint right_ankle_pitch: axis 0 0 1 -> 0 1 0; origin xyz=0.093 0 0 rpy=3.14159 0 0 -> xyz=0 0 -0.093 rpy=0 0 0
- joint right_ankle_roll: axis 0 0 1 -> 1 0 0; origin xyz=0 0 0 rpy=-1.5707963 0 0 -> xyz=0 0 0 rpy=0 0 0
- joint right_elbow_pitch: axis 0 0 1 -> 0 1 0 ; origin xyz=-0.06 0 0.016 rpy=-1.5707963 3.14159 0 -> xyz=-0.016 0 -0.06  rpy=0 0 0
- joint right_hip_pitch: axis 0 0 1 -> 0 1 0; origin xyz=0 0 0 rpy=1.5707963 0 -1.5707963 -> xyz=0 0 0 rpy=0 0 0
- joint right_hip_roll: axis 0 0 1 -> 1 0 0; origin xyz=0 0 0.028652 rpy=-1.5707963 0 0 -> xyz=0 0 -0.028652 rpy=0 0 0
- joint right_hip_yaw: origin xyz=-0.005 -0.037 -0.09355 rpy=0 3.14159 1.5707963 -> xyz=-0.005 -0.037 -0.09355 rpy=0 0 0
- joint right_knee_pitch: axis 0 0 1 -> 0 1 0; origin xyz=0.093 0 0 rpy=0 0 0 -> xyz=0 0 -0.093 rpy=0 0 0
- joint right_shoulder_pitch: axis 0 0 1 -> 0 1 0; origin xyz=0 0 0 rpy=0 0 -1.5707963 -> xyz=0 0 0 rpy=0 0 0
- joint right_shoulder_roll: axis 0 0 1 -> 1 0 0; origin xyz=0.016 0 0.02165 rpy=-1.5707963 1.5707963 0 -> xyz=0 -0.02165 -0.016 rpy=0 0 0
