Commit message: darwin now has a head :moyai:

File: colcon_ws/src/robots/darwin/darwin_description/urdf/darwin_lab.urdf (robot description, URDF)
Before this commit: robot darwin_lab, 31 links, 30 joints
Links:
- added link camera_optical; collision box size=0.032 0.005 0.032; visual box size=0.032 0.005 0.032
- link neck_link: mass None -> 0.024357719
Joints:
- added joint camera_joint: type fixed, parent head_link, child camera_optical, origin xyz=0 0 0.0235 rpy=0 0 0
